File: Hardware/UnnamedClockProject/UnnamedClockProject.kicad_sch (KiCad schematic)
At the start: 34 parts, among them J101 CLOCK_OUT, J102 POWER, J103 BUTTONS, Q101 2N3904, U104 G3MB-202P, U105 G3MB-202P, U106 G3MB-202P, U107 CAT24C256

Commit message: Boilerplate new file upstream
Parts:
- U104, U105, U106: footprint OptoDevice:Finder_34.81 -> ac1ja:OptoRelay
Changed lines of the file:
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@@
       (effects (font (size 1.27 1.27)))
     )
-    (property "Footprint" "OptoDevice:Finder_34.81" (at 146.685 29.21 0)
+    (property "Footprint" "ac1ja:OptoRelay" (at 146.685 29.21 0)
       (effects (font (size 1.27 1.27) italic) (justify left) hide)
     )
@@
       (effects (font (size 1.27 1.27)))
     )
-    (property "Footprint" "OptoDevice:Finder_34.81" (at 146.685 46.355 0)
+    (property "Footprint" "ac1ja:OptoRelay" (at 146.685 46.355 0)
       (effects (font (size 1.27 1.27) italic) (justify left) hide)
     )
@@
       (effects (font (size 1.27 1.27)))
     )
-    (property "Footprint" "OptoDevice:Finder_34.81" (at 146.685 64.77 0)
+    (property "Footprint" "ac1ja:OptoRelay" (at 146.685 64.77 0)
       (effects (font (size 1.27 1.27) italic) (justify left) hide)
     )
